Commit message: added segment 3

File: grab_it_gz/model/xacro/grab_it.xacro (robot description, xacro)
@@ -13,6 +13,6 @@
             <origin xyz="0 0 0" rpy="0 0 0"/>
             <inertial>
-                <mass value="10.0"/>
-                <inertia ixx="0" ixy="0" ixz="0" iyy="0.001" iyz="0.001" izz="0.001"/>
+                <mass value="1.0"/>
+                <inertia ixx="0.01" ixy="0" ixz="0" iyy="0.01" iyz="0" izz="0.01"/>
             </inertial>
             <visual name="${name}_base_link">
@@ -32,6 +32,6 @@
             <origin xyz="0 0 0" rpy="0 0 0"/>
             <inertial>
-                <mass value="1"/>
-                <inertia ixx="0.001" ixy="0.001" ixz="0.001" iyy="0.001" iyz="0.001" izz="0.001"/>
+                <mass value="1.0"/>
+                <inertia ixx="0.01" ixy="0.0" ixz="0.0" iyy="0.01" iyz="0.0" izz="0.01"/>
             </inertial>
             <!-- Visuals -->
@@ -53,6 +53,6 @@
             <origin xyz="0 0 0" rpy="0 0 0"/>
             <inertial>
-                <mass value="1"/>
-                <inertia ixx="0.001" ixy="0.001" ixz="0.001" iyy="0.001" iyz="0.001" izz="0.001"/>
+                <mass value="1.0"/>
+                <inertia ixx="0.01" ixy="0.0" ixz="0.0" iyy="0.01" iyz="0.0" izz="0.01"/>
             </inertial>
             <!-- Visuals -->
@@ -67,4 +67,25 @@
                 <geometry>
                     <mesh filename="model://meshes/AXIS_2.dae"/>
+                </geometry>
+            </collision>
+        </link>
+        <!-- link_3 -->
+        <link name="${name}_link_3">
+            <origin xyz="0 0 0" rpy="0 0 0"/>
+            <inertial>
+                <mass value="1.0"/>
+                <inertia ixx="0.01" ixy="0.0" ixz="0.0" iyy="0.01" iyz="0.0" izz="0.01"/>
+            </inertial>
+            <!-- Visuals -->
+            <visual name='l3_e_1_visual'>
+                <geometry>
+                    <mesh filename="model://meshes/AXIS_3.dae"/>
+                </geometry>
+                <material name="material_silber"/>
+            </visual>
+            <!-- Collisions -->
+            <collision name='l3_e_1_collision'>
+                <geometry>
+                    <mesh filename="model://meshes/AXIS_3.dae"/>
                 </geometry>
             </collision>
@@ -86,4 +107,12 @@
             <dynamics damping="0.1"/>
         </joint>
+        <joint name='joint_3' type='revolute'>
+            <origin xyz="-0.0475 0.002 0.11125" rpy="0 0 0"/>
+            <parent link="${name}_link_2"/>
+            <child link="${name}_link_3"/>
+            <axis xyz ="1 0 0"/>
+            <limit lower="-3.01941960595019" upper="3.01941960595019" velocity="3" effort="50"/>
+            <dynamics damping="0.1"/>
+        </joint>
         <ros2_control name="GazeboSimSystem" type="system">
             <hardware>
@@ -92,10 +121,21 @@
             <joint name="joint_1">
                 <command_interface name="position"/>
-                <state_interface name="position"/>
+                <state_interface name="position">
+                    <param name="initial_value">0.0</param>
+                </state_interface>
                 <state_interface name="velocity"/>
             </joint>
             <joint name="joint_2">
                 <command_interface name="position"/>
-                <state_interface name="position"/>
+                <state_interface name="position">
+                    <param name="initial_value">0.0</param>
+                </state_interface>
+                <state_interface name="velocity"/>
+            </joint>
+            <joint name="joint_3">
+                <command_interface name="position"/>
+                <state_interface name="position">
+                    <param name="initial_value">0.0</param>
+                </state_interface>
                 <state_interface name="velocity"/>
             </joint>

Commit message: added segment 4

File: grab_it_gz/model/xacro/grab_it.xacro (robot description, xacro)
@@ -91,4 +91,25 @@
             </collision>
         </link>
+        <!-- link_4 -->
+        <link name="${name}_link_4">
+            <origin xyz="0 0 0" rpy="0 0 0"/>
+            <inertial>
+                <mass value="1.0"/>
+                <inertia ixx="0.01" ixy="0.0" ixz="0.0" iyy="0.01" iyz="0.0" izz="0.01"/>
+            </inertial>
+            <!-- Visuals -->
+            <visual name='l4_e_1_visual'>
+                <geometry>
+                    <mesh filename="model://meshes/AXIS_4.dae"/>
+                </geometry>
+                <material name="material_silber"/>
+            </visual>
+            <!-- Collisions -->
+            <collision name='l4_e_1_collision'>
+                <geometry>
+                    <mesh filename="model://meshes/AXIS_4.dae"/>
+                </geometry>
+            </collision>
+        </link>
         <joint name='joint_1' type='revolute'>
             <origin xyz="0 0.0625 0.0725" rpy="0 0 0"/>
@@ -108,7 +129,15 @@
         </joint>
         <joint name='joint_3' type='revolute'>
-            <origin xyz="-0.0475 0.002 0.11125" rpy="0 0 0"/>
+            <origin xyz="-0.0475 0.002 0.10125" rpy="0 0 0"/>
             <parent link="${name}_link_2"/>
             <child link="${name}_link_3"/>
+            <axis xyz ="1 0 0"/>
+            <limit lower="-3.01941960595019" upper="3.01941960595019" velocity="3" effort="50"/>
+            <dynamics damping="0.1"/>
+        </joint>
+        <joint name='joint_4' type='revolute'>
+            <origin xyz="-0.00434 -0.01 0.10625" rpy="0 0 0"/>
+            <parent link="${name}_link_3"/>
+            <child link="${name}_link_4"/>
             <axis xyz ="1 0 0"/>
             <limit lower="-3.01941960595019" upper="3.01941960595019" velocity="3" effort="50"/>
@@ -140,4 +169,11 @@
                 <state_interface name="velocity"/>
             </joint>
+            <joint name="joint_4">
+                <command_interface name="position"/>
+                <state_interface name="position">
+                    <param name="initial_value">0.0</param>
+                </state_interface>
+                <state_interface name="velocity"/>
+            </joint>
         </ros2_control>
     </xacro:macro>

Commit message: added axis 5 (flange)

File: grab_it_gz/model/xacro/grab_it.xacro (robot description, xacro)
@@ -112,4 +112,25 @@
             </collision>
         </link>
+        <!-- link_5 -->
+        <link name="${name}_link_5">
+            <origin xyz="0 0 0" rpy="0 0 0"/>
+            <inertial>
+                <mass value="1.0"/>
+                <inertia ixx="0.01" ixy="0.0" ixz="0.0" iyy="0.01" iyz="0.0" izz="0.01"/>
+            </inertial>
+            <!-- Visuals -->
+            <visual name='l5_e_1_visual'>
+                <geometry>
+                    <mesh filename="model://meshes/AXIS_5.dae"/>
+                </geometry>
+                <material name="material_silber"/>
+            </visual>
+            <!-- Collisions -->
+            <collision name='l5_e_1_collision'>
+                <geometry>
+                    <mesh filename="model://meshes/AXIS_5.dae"/>
+                </geometry>
+            </collision>
+        </link>
         <joint name='joint_1' type='revolute'>
             <origin xyz="0 0.0625 0.0725" rpy="0 0 0"/>
@@ -144,4 +165,12 @@
             <dynamics damping="0.1"/>
         </joint>
+        <joint name='joint_5' type='revolute'>
+            <origin xyz="0.025 0.02 0.042625" rpy="0 0 0"/>
+            <parent link="${name}_link_4"/>
+            <child link="${name}_link_5"/>
+            <axis xyz ="0 0 1"/>
+            <limit lower="-3.01941960595019" upper="3.01941960595019" velocity="3" effort="50"/>
+            <dynamics damping="0.1"/>
+        </joint>
         <ros2_control name="GazeboSimSystem" type="system">
             <hardware>
@@ -176,4 +205,11 @@
                 <state_interface name="velocity"/>
             </joint>
+            <joint name="joint_5">
+                <command_interface name="position"/>
+                <state_interface name="position">
+                    <param name="initial_value">0.0</param>
+                </state_interface>
+                <state_interface name="velocity"/>
+            </joint>
         </ros2_control>
     </xacro:macro>
